File: hardware/openkey-cps2.kicad_pcb (KiCad board)
At the start: 2 copper layers, 23.3 x 23 mm, 14 parts, among them CN9 Conn_01x06, J1 Solder Pad, U1 ATtinyxx4

Commit message: Some minor tweaks around the vcc jumper and pad
Should make it more obvious what is for what
Parts:
- moved J1 10.8 mm to (137.2, 104.8)
- moved JP9 1.96 mm to (136.7, 97.4)
Routing:
- net VCC: track 13.6 -> 16.3 mm
- net GND: track 50.0 -> 50.9 mm
- net /CN9 VCC: track 20.8 -> 20.0 mm
Changed lines of the file:
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@@
     (property "Sheetname" "")
     (attr through_hole)
-    (fp_text reference "CN9" (at 2.45 6.47 90) (layer "F.SilkS")
+    (fp_text reference "CN9" (at 2.45 6.405 90) (layer "F.SilkS")
       (effects (font (size 1 1) (thickness 0.15)))
     )
@@
   )
   (footprint "Jumper:SolderJumper-2_P1.3mm_Open_RoundedPad1.0x1.5mm" (layer "F.Cu")
-    (at 136.64 99.34)
+    (at 136.7 97.38)
     (descr "SMD Solder Jumper, 1x1.5mm, rounded Pads, 0.3mm gap, open")
     (tags "solder jumper open")
@@
   )
   (footprint "TestPoint:TestPoint_Pad_D2.5mm" (layer "F.Cu")
-    (at 136.79 94.03)
+    (at 137.18 104.81)
     (descr "SMD pad as test Point, diameter 2.5mm")
     (tags "test point SMD pad")
@@
       (effects (font (size 1 1) (thickness 0.15)))
     )
-    (fp_text value "ATtinyxx4" (at 0.16 0.11 180 unlocked) (layer "F.SilkS")
+    (fp_text value "ATtinyxx4" (at 0.06 0.11 180 unlocked) (layer "F.SilkS")
       (effects (font (size 1 1) (thickness 0.15)))
     )
@@
       ) (layer "B.SilkS") (width 0.01) (fill solid))
   )
+  (gr_rect (start 132.93 101.37) (end 139.03 108.08) (layer "F.SilkS") (width 0.15) (fill none))
+  (gr_rect (start 134.58 88.23) (end 139.04 99.09) (layer "F.SilkS") (width 0.15) (fill none))
   (gr_rect (start 116.4 85.8) (end 139.7 108.775) (layer "Edge.Cuts") (width 0.1) (fill none))
   (gr_text "6" (at 117.8 90.85 90) (layer "B.SilkS")
@@
     (effects (font (size 1 1) (thickness 0.15)) (justify mirror))
   )
-  (gr_text "93646B-6/7\nVCC Jumper" (at 136.81 104.61 90) (layer "F.SilkS")
+  (gr_text "93646B-6/7\nVCC Jumper" (at 136.8 92.29 90) (layer "F.SilkS")
     (effects (font (size 0.7 0.7) (thickness 0.12)))
   )
@@
     (effects (font (size 1 1) (thickness 0.15)))
   )
-  (gr_text "HW REV ${REV}" (at 127.6 107.675) (layer "F.SilkS")
+  (gr_text "HW REV ${REV}" (at 126.37 107.74) (layer "F.SilkS")
     (effects (font (size 0.7 0.7) (thickness 0.1)))
   )
@@
     (effects (font (size 1 1) (thickness 0.15)))
   )
-  (gr_text "93646B-5\nVCC Pad" (at 136.9 89.25 90) (layer "F.SilkS")
+  (gr_text "93646B-5\nVCC Pad" (at 134.48 104.72 90) (layer "F.SilkS")
     (effects (font (size 0.7 0.7) (thickness 0.12)))
   )
-  (gr_text "OPENKEY CPS2" (at 127.6 87.025) (layer "F.SilkS")
+  (gr_text "OPENKEY CPS2" (at 127.63 87.025) (layer "F.SilkS")
     (effects (font (size 1 1) (thickness 0.15)))
   )
@@
     (effects (font (size 0.7 0.7) (thickness 0.1)))
   )
-  (segment (start 135.2575 94.03) (end 136.79 94.03) (width 0.25) (layer "F.Cu") (net 1))
+  (segment (start 137.35 104.64) (end 137.18 104.81) (width 0.25) (layer "F.Cu") (net 1))
+  (segment (start 136.98 96.24) (end 137.35 96.61) (width 0.25) (layer "F.Cu") (net 1))
+  (segment (start 137.35 96.61) (end 137.35 97.38) (width 0.25) (layer "F.Cu") (net 1))
   (segment (start 130.61 94.825) (end 130.61 95.59) (width 0.25) (layer "F.Cu") (net 1))
-  (segment (start 137.29 99.34) (end 137.29 97.08) (width 0.25) (layer "F.Cu") (net 1))
+  (segment (start 133.0525 96.24) (end 136.98 96.24) (width 0.25) (layer "F.Cu") (net 1))
   (segment (start 131.2575 96.2375) (end 133.05 96.2375) (width 0.25) (layer "F.Cu") (net 1))
-  (segment (start 133.05 96.2375) (end 135.2575 94.03) (width 0.25) (layer "F.Cu") (net 1))
-  (segment (start 137.29 97.08) (end 136.79 96.58) (width 0.25) (layer "F.Cu") (net 1))
   (segment (start 130.61 95.59) (end 131.2575 96.2375) (width 0.25) (layer "F.Cu") (net 1))
-  (segment (start 136.79 96.58) (end 136.79 94.03) (width 0.25) (layer "F.Cu") (net 1))
+  (segment (start 137.35 97.26) (end 137.35 104.64) (width 0.25) (layer "F.Cu") (net 1))
   (segment (start 118.55 104.85) (end 118.55 104.66) (width 0.25) (layer "F.Cu") (net 2))
   (segment (start 121.775 90.125) (end 123.8 90.125) (width 0.25) (layer "F.Cu") (net 2))
-  (segment (start 133.05 104.325) (end 132.9 104.475) (width 0.25) (layer "F.Cu") (net 2))
   (segment (start 126.35 90.125) (end 131.45 90.125) (width 0.25) (layer "F.Cu") (net 2))
   (segment (start 123.8 104.475) (end 122.625 104.475) (width 0.25) (layer "F.Cu") (net 2))
-  (segment (start 133.05 99.75) (end 133.05 104.325) (width 0.25) (layer "F.Cu") (net 2))
+  (segment (start 131.2675 98.3125) (end 130.61 98.97) (width 0.25) (layer "F.Cu") (net 2))
   (segment (start 122.625 104.475) (end 121.83 105.27) (width 0.25) (layer "F.Cu") (net 2))
   (segment (start 128.9 104.475) (end 126.35 104.475) (width 0.25) (layer "F.Cu") (net 2))
   (segment (start 118.55 104.66) (end 118.55 92.32) (width 0.25) (layer "F.Cu") (net 2))
   (segment (start 132.9 104.475) (end 131.45 104.475) (width 0.25) (layer "F.Cu") (net 2))
-  (segment (start 133.025 99.775) (end 133.05 99.75) (width 0.25) (layer "F.Cu") (net 2))
+  (segment (start 133.05 98.3125) (end 131.2675 98.3125) (width 0.25) (layer "F.Cu") (net 2))
   (segment (start 118.55 92.32) (end 119.925 90.945) (width 0.25) (layer "F.Cu") (net 2))
-  (segment (start 130.61 99.775) (end 133.025 99.775) (width 0.25) (layer "F.Cu") (net 2))
+  (segment (start 133.05 104.325) (end 132.9 104.475) (width 0.25) (layer "F.Cu") (net 2))
   (segment (start 121.83 105.27) (end 118.97 105.27) (width 0.25) (layer "F.Cu") (net 2))
-  (segment (start 133.05 98.225) (end 133.05 99.75) (width 0.25) (layer "F.Cu") (net 2))
   (segment (start 119.925 90.945) (end 120.955 90.945) (width 0.25) (layer "F.Cu") (net 2))
   (segment (start 131.45 104.475) (end 128.9 104.475) (width 0.25) (layer "F.Cu") (net 2))
@@
   (segment (start 123.8 90.125) (end 126.35 90.125) (width 0.25) (layer "F.Cu") (net 2))
   (segment (start 120.955 90.945) (end 121.775 90.125) (width 0.25) (layer "F.Cu") (net 2))
+  (segment (start 130.61 98.97) (end 130.61 99.775) (width 0.25) (layer "F.Cu") (net 2))
+  (segment (start 133.05 98.3125) (end 133.05 104.325) (width 0.25) (layer "F.Cu") (net 2))
   (segment (start 118.97 105.27) (end 118.55 104.85) (width 0.25) (layer "F.Cu") (net 2))
   (segment (start 124.26 100.89) (end 124.26 99.775) (width 0.25) (layer "F.Cu") (net 3))
@@
   (segment (start 125.53 101.145) (end 124.65 102.025) (width 0.25) (layer "F.Cu") (net 14))
   (segment (start 125.53 101.145) (end 125.53 99.775) (width 0.25) (layer "F.Cu") (net 14))
+  (segment (start 123.04 101.56) (end 124.226396 101.56) (width 0.25) (layer "F.Cu") (net 15))
   (segment (start 120.955 103.645) (end 123.04 101.56) (width 0.25) (layer "F.Cu") (net 15))
+  (segment (start 124.885 98.773249) (end 126.398248 97.26) (width 0.25) (layer "F.Cu") (net 15))
   (segment (start 124.226396 101.56) (end 124.885 100.901396) (width 0.25) (layer "F.Cu") (net 15))
   (segment (start 119.925 103.645) (end 120.955 103.645) (width 0.25) (layer "F.Cu") (net 15))
-  (segment (start 123.04 101.56) (end 124.226396 101.56) (width 0.25) (layer "F.Cu") (net 15))
+  (segment (start 126.398248 97.26) (end 136.05 97.26) (width 0.25) (layer "F.Cu") (net 15))
   (segment (start 124.885 100.901396) (end 124.885 98.773249) (width 0.25) (layer "F.Cu") (net 15))
-  (segment (start 133.91 97.26) (end 135.99 99.34) (width 0.25) (layer "F.Cu") (net 15))
-  (segment (start 124.885 98.773249) (end 126.398248 97.26) (width 0.25) (layer "F.Cu") (net 15))
-  (segment (start 126.398248 97.26) (end 133.91 97.26) (width 0.25) (layer "F.Cu") (net 15))
 )
